File: pcb/rcs-controller.kicad_pcb (KiCad board)
At the start: 2 copper layers, 1 part

Commit message: First circuit board
Parts:
- removed REF**: FeatherS3, Additional_parts:FeatherS3
- added C1: 10u, Capacitor_SMD:C_0805_2012Metric, F.Cu at (67.2, 20.8)
- added C10: 100n, Capacitor_SMD:C_0603_1608Metric, F.Cu at (52.7, 10.6)
- added C11: 2.2n, Capacitor_SMD:C_0603_1608Metric, F.Cu at (52.7, 13.1)
- added C12: 10u, Capacitor_SMD:C_0603_1608Metric, F.Cu at (52.7, 15.6)
- added C13: 2.2n, Capacitor_SMD:C_0603_1608Metric, F.Cu at (52.7, 18.1)
- added C14: 22u, Capacitor_SMD:C_0805_2012Metric, F.Cu at (67.2, 35.9)
- added C15: 22u, Capacitor_SMD:C_0805_2012Metric, F.Cu at (67.2, 38.9)
- added C16: 22u, Capacitor_SMD:C_0805_2012Metric, F.Cu at (67.2, 41.9)
- added C17: 100n, Capacitor_SMD:C_0603_1608Metric, F.Cu at (34.6, 26.4)
- added C18: 100n, Capacitor_SMD:C_0603_1608Metric, F.Cu at (34.6, 28.9)
- added C19: 100n, Capacitor_SMD:C_0603_1608Metric, F.Cu at (34.6, 31.4)
- added C2: 10u, Capacitor_SMD:C_0805_2012Metric, F.Cu at (67.2, 23.9)
- added C20: 100n, Capacitor_SMD:C_0603_1608Metric, F.Cu at (34.6, 33.9)
- added C26: 1n, Capacitor_SMD:C_0603_1608Metric, F.Cu at (56.7, 3.02)
- added C29: 100n, Capacitor_SMD:C_0603_1608Metric, F.Cu at (56.7, 5.53)
- added C4: 10u, Capacitor_SMD:C_0805_2012Metric, F.Cu at (67.2, 26.9)
- added C5: 10u, Capacitor_SMD:C_0603_1608Metric, F.Cu at (52.7, 3.02)
- added C6: 10u, Capacitor_SMD:C_0805_2012Metric, F.Cu at (67.2, 29.9)
- added C7: 100n, Capacitor_SMD:C_0603_1608Metric, F.Cu at (52.7, 5.53)
- added C8: 10u, Capacitor_SMD:C_0805_2012Metric, F.Cu at (67.2, 32.9)
- added C9: 100n, Capacitor_SMD:C_0603_1608Metric, F.Cu at (52.7, 8.04)
- added D1: GRN, LED_SMD:LED_0603_1608Metric, F.Cu at (86.1, 3.06)
- added D10: RBR5L30BDDTE25, Diode_SMD:D_SMA, F.Cu at (36.7, 39.9)
- added D11: RBR5L30BDDTE25, Diode_SMD:D_SMA, F.Cu at (36.7, 44.5)
- added D2: GRN, LED_SMD:LED_0603_1608Metric, F.Cu at (86.1, 5.65)
- added D4: RBR5L30BDDTE25, Diode_SMD:D_SMA, F.Cu at (81.0, 29.5)
- added D5: GRN, LED_SMD:LED_0603_1608Metric, F.Cu at (86.1, 8.24)
- added D6: LED, LED_SMD:LED_0603_1608Metric, F.Cu at (34.7, 48.1)
- added D7: GRN, LED_SMD:LED_0603_1608Metric, F.Cu at (86.1, 10.8)
- added D8: LED, LED_SMD:LED_0603_1608Metric, F.Cu at (34.7, 50.6)
- added D9: RBR5L30BDDTE25, Diode_SMD:D_SMA, F.Cu at (81.0, 34.0)
- added J1: 00222-32051, Connector_Molex:Molex_KK-254_AE-6410-06A_1x06_P2.54mm_Vertical, F.Cu at (69.0, 5.71)
- added J10: 0022-232021, Connector_Molex:Molex_KK-254_AE-6410-02A_1x02_P2.54mm_Vertical, F.Cu at (60.1, 23.3)
- added J2: 0022-232021, Connector_Molex:Molex_KK-254_AE-6410-02A_1x02_P2.54mm_Vertical, F.Cu at (53.0, 23.3)
- added J3: 0022-232041, Connector_Molex:Molex_KK-254_AE-6410-04A_1x04_P2.54mm_Vertical, F.Cu at (71.7, 23.3)
- added J4: Screw_Terminal_4_P3.50mm, TerminalBlock_Phoenix:TerminalBlock_Phoenix_PT-1,5-4-3.5-H_1x04_P3.50mm_Horizontal, F.Cu at (35.4, 5.89)
- added J8: 00222-32051, Connector_Molex:Molex_KK-254_AE-6410-06A_1x06_P2.54mm_Vertical, F.Cu at (69.0, 13.6)
- added L1: 1.5uH, Inductor_SMD:L_Vishay_IHLP-2020, F.Cu at (54.9, 30.5)
- added L2: 4.7uH, Inductor_SMD:L_Vishay_IHLP-2020, F.Cu at (54.9, 37.2)
- added Q1: SI7465DP-T1-E3, PCM_Package_SON_AKL:Infineon_PG-TDSON-8, F.Cu at (81.1, 39.6)
- added Q2: SI7465DP-T1-E3, PCM_Package_SON_AKL:Infineon_PG-TDSON-8, F.Cu at (36.8, 15.0)
- added Q3: SI7465DP-T1-E3, PCM_Package_SON_AKL:Infineon_PG-TDSON-8, F.Cu at (36.8, 21.8)
- added Q4: PMV45EN2, PCM_Package_TO_SOT_SMD_AKL:SOT-23, F.Cu at (43.0, 27.5)
- added Q5: PMV45EN2, PCM_Package_TO_SOT_SMD_AKL:SOT-23, F.Cu at (43.0, 32.2)
- added R1: 10k, Resistor_SMD:R_0603_1608Metric, F.Cu at (56.7, 8.04)
- added R10: 150k, Resistor_SMD:R_0603_1608Metric, F.Cu at (60.7, 8.04)
- added R11: 2.4k, Resistor_SMD:R_0603_1608Metric, F.Cu at (60.7, 10.6)
- added R12: 750, Resistor_SMD:R_0603_1608Metric, F.Cu at (60.7, 13.1)
- added R13: 100m, Resistor_SMD:R_1206_3216Metric, F.Cu at (61.8, 28.8)
- added R14: 1k, Resistor_SMD:R_0603_1608Metric, F.Cu at (60.7, 15.6)
- added R15: 1k, Resistor_SMD:R_0603_1608Metric, F.Cu at (60.7, 18.1)
- added R16: 4.7k, Resistor_SMD:R_0603_1608Metric, F.Cu at (64.7, 3.02)
- added R17: 150k, Resistor_SMD:R_0603_1608Metric, F.Cu at (64.7, 5.53)
- added R18: 10k, Resistor_SMD:R_0603_1608Metric, F.Cu at (64.7, 8.04)
- added R19: 33k, Resistor_SMD:R_0603_1608Metric, F.Cu at (64.7, 10.6)
- added R2: 4.7k, Resistor_SMD:R_0603_1608Metric, F.Cu at (56.7, 10.6)
- added R20: 10k, Resistor_SMD:R_0603_1608Metric, F.Cu at (64.7, 13.1)
- added R21: 10k, Resistor_SMD:R_0603_1608Metric, F.Cu at (38.6, 26.4)
- added R22: 10k, Resistor_SMD:R_0603_1608Metric, F.Cu at (38.6, 28.9)
- added R23: 10k, Resistor_SMD:R_0603_1608Metric, F.Cu at (38.6, 31.4)
- added R24: 1k, Resistor_SMD:R_0603_1608Metric, F.Cu at (38.6, 33.9)
- added R25: 1k, Resistor_SMD:R_0603_1608Metric, F.Cu at (38.6, 36.4)
- added R3: 4.7k, Resistor_SMD:R_0603_1608Metric, F.Cu at (56.7, 13.1)
- added R35: 60.4, Resistor_SMD:R_1206_3216Metric, F.Cu at (61.8, 32.1)
- added R36: 60.4, Resistor_SMD:R_1206_3216Metric, F.Cu at (61.8, 35.4)
- added R4: 10k, Resistor_SMD:R_0603_1608Metric, F.Cu at (56.7, 15.6)
- added R5: 10k, Resistor_SMD:R_0603_1608Metric, F.Cu at (56.7, 18.1)
- added R6: 10k, Resistor_SMD:R_0603_1608Metric, F.Cu at (60.7, 3.02)
- added R8: 10k, Resistor_SMD:R_0603_1608Metric, F.Cu at (34.6, 36.4)
- added R9: 470k, Resistor_SMD:R_0603_1608Metric, F.Cu at (60.7, 5.53)
- added TP1: Test-Point, psas-footprints:TP-through-hole-1X01, F.Cu at (70.7, 28.4)
- added TP2: Test-Point, psas-footprints:TP-through-hole-1X01, F.Cu at (70.7, 31.0)
- added TP3: Test-Point, psas-footprints:TP-through-hole-1X01, F.Cu at (70.7, 33.5)
- added TP30: Test-Point, psas-footprints:TP-through-hole-1X01, F.Cu at (75.7, 28.4)
- added TP31: Test-Point, psas-footprints:TP-through-hole-1X01, F.Cu at (75.7, 31.0)
- added TP32: Test-Point, psas-footprints:TP-through-hole-1X01, F.Cu at (75.7, 33.5)
- added TP4: Test-Point, psas-footprints:TP-through-hole-1X01, F.Cu at (70.7, 36.0)
- added TP5: Test-Point, psas-footprints:TP-through-hole-1X01, F.Cu at (73.2, 28.4)
- added TP6: Test-Point, psas-footprints:TP-through-hole-1X01, F.Cu at (73.2, 31.0)
- added TP7: Test-Point, psas-footprints:TP-through-hole-1X01, F.Cu at (73.2, 33.5)
- added TP9: Test-Point, psas-footprints:TP-through-hole-1X01, F.Cu at (73.2, 36.0)
- added U1: LSM6DSOX, Package_LGA:LGA-14_3x2.5mm_P0.5mm_LayoutBorder3x4y, F.Cu at (43.0, 39.8)
- added U2: MP26123DR-LF-Z, Package_DFN_QFN:QFN-16-1EP_4x4mm_P0.65mm_EP2.5x2.5mm, F.Cu at (84.7, 22.5)
- added U3: TPS63070, psas-footprints:U-TI-TPS63070, F.Cu at (61.2, 39.0)
- added U4: FeatherS3, Module:Adafruit_Feather, F.Cu at (10.3, 8.89)
Routing:
- added copper zone on B.Cu, net GND
- added copper zone on F.Cu, net GND
Other:
- board outline added: 100 x 75 mm

Commit message: Push to move to other machine
Parts:
- removed C26: 1n, Capacitor_SMD:C_0603_1608Metric
- removed R35, R36: 60.4, Resistor_SMD:R_1206_3216Metric
- moved J4 187.9 mm to (176.5, 130.0)
- moved J10 172.0 mm to (195.0, 130.0)
- moved R15 168.6 mm to (195.0, 120.0), turned to 90 degrees
- moved R14 166.7 mm to (190.0, 120.8), turned to 90 degrees
- moved C9 161.1 mm to (184.2, 101.1)
- moved C10 161.1 mm to (189.2, 96.1)
- moved C13 159.3 mm to (194.2, 91.1)
- moved Q3 158.7 mm to (162.9, 118.1)
- moved R12 157.1 mm to (190.8, 101.1)
- moved R24 156.2 mm to (175.0, 110.0), turned to 90 degrees
- moved C1 155.7 mm to (194.1, 111.1)
- moved D8 154.4 mm to (175.0, 115.0), turned to 90 degrees
- moved D11 154.2 mm to (165.0, 130.0), turned to -90 degrees
- moved R22 154.2 mm to (155.0, 130.0), turned to 90 degrees
- moved R11 153.3 mm to (190.8, 91.5)
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Routing:
- net GND: track 0.00 -> 530.2 mm, vias 0 -> 42
- net +3.3V: track 0.00 -> 306.5 mm, vias 0 -> 7
- net VBUS: track 0.00 -> 285.0 mm, vias 0 -> 11
- net +BATT: track 0.00 -> 243.3 mm, vias 0 -> 16
- net CANH: track 0.00 -> 177.3 mm, vias 0 -> 9
- net UMB_~{ON}: track 0.00 -> 171.5 mm, vias 0 -> 6
- net /Power/VUMB: track 0.00 -> 170.8 mm, vias 0 -> 4
- net Net-(Q2-G): track 0.00 -> 159.9 mm, vias 0 -> 13
- net Net-(D11-K): track 0.00 -> 149.1 mm, vias 0 -> 6
- net BATT_READ: track 0.00 -> 145.2 mm, vias 0 -> 6
- net Net-(Q1-G): track 0.00 -> 123.9 mm, vias 0 -> 8
- net Net-(U3-L2): track 0.00 -> 111.3 mm, vias 0 -> 8
- net Net-(U3-VAUX): track 0.00 -> 105.7 mm, vias 0 -> 3
- net Net-(D8-K): track 0.00 -> 94.8 mm, vias 0 -> 6
- net Net-(Q5-G): track 0.00 -> 93.0 mm, vias 0 -> 4
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
Commit message: Rev2
Parts:
- moved J10 63.3 mm to (133.6, 145.3)
- moved R15 61.3 mm to (137.2, 140.4)
- moved R14 60.6 mm to (132.6, 140.4)
- moved J4 59.1 mm to (119.0, 143.7)
- moved C1 53.1 mm to (143.8, 94.0), turned to 180 degrees
- moved C13 52.8 mm to (146.0, 112.6), turned to 180 degrees
- moved C4 48.6 mm to (117.1, 114.8), turned to -90 degrees
- moved R10 48.5 mm to (132.2, 117.7), turned to -90 degrees
- moved C2 47.0 mm to (113.9, 114.7), turned to -90 degrees
- moved R9 46.7 mm to (132.2, 114.7), turned to -90 degrees
- moved R11 45.6 mm to (149.0, 109.8), turned to 180 degrees
- moved TP2 45.2 mm to (136.1, 86.2)
- moved R12 43.4 mm to (149.0, 112.6), turned to 180 degrees
- moved TP4 43.0 mm to (151.2, 94.5)
- moved R16 42.9 mm to (145.5, 117.9), turned to -90 degrees
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Routing:
- net GND: track 530.2 -> 349.0 mm, vias 42 -> 27
- net VBUS: track 285.0 -> 103.9 mm, vias 11 -> 1
- net +3.3V: track 306.5 -> 140.1 mm, vias 7 -> 4
- net CANH: track 177.3 -> 26.4 mm, vias 9 -> 0
- net Net-(Q2-G): track 159.9 -> 9.33 mm, vias 13 -> 0
- net +BATT: track 243.3 -> 117.7 mm, vias 16 -> 2
- net BATT_READ: track 145.2 -> 31.6 mm, vias 6 -> 0
- net Net-(D11-K): track 149.1 -> 37.5 mm, vias 6 -> 0
- net UMB_~{ON}: track 171.5 -> 63.1 mm, vias 6 -> 2
- net /Power/VUMB: track 170.8 -> 64.6 mm, vias 4 -> 1
- net Net-(U3-L2): track 111.3 -> 6.21 mm, vias 8 -> 0
- net Net-(U3-VAUX): track 105.7 -> 2.30 mm, vias 3 -> 0
- net Net-(D8-K): track 94.8 -> 3.68 mm, vias 6 -> 0
- net Net-(C13-Pad1): track 87.3 -> 1.40 mm, vias 7 -> 0
- net Net-(U3-L1): track 88.6 -> 6.04 mm, vias 3 -> 0
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
Commit message: Submit for review 4.23.2025
Parts:
- removed C12, C5: 10u, Capacitor_SMD:C_0603_1608Metric
- removed D6, D8: LED, LED_SMD:LED_0603_1608Metric
- removed TP9: Test-Point, psas-footprints:TP-through-hole-1X01
- added C26: 1n, Capacitor_SMD:C_0603_1608Metric, F.Cu at (149.8, 90.3)
- added LED1: LED_0603_Amber, PCM_LED_SMD_AKL:LED_0603_1608Metric, F.Cu at (132.8, 136.7)
- added LED2: LED_0603_Amber, PCM_LED_SMD_AKL:LED_0603_1608Metric, F.Cu at (112.1, 139.5)
- added R26: 10k, Resistor_SMD:R_0603_1608Metric, F.Cu at (120.2, 108.0)
- added R27: 10k, Resistor_SMD:R_0603_1608Metric, F.Cu at (125.7, 110.1)
- added R35: 60.4, Resistor_SMD:R_1206_3216Metric, F.Cu at (147.5, 86.1)
- added R36: 60.4, Resistor_SMD:R_1206_3216Metric, F.Cu at (150.5, 88.4)
- added TP33: Test-Point, psas-footprints:TP-through-hole-1X01, F.Cu at (118.1, 109.7)
- added TP34: Test-Point, psas-footprints:TP-through-hole-1X01, F.Cu at (122.5, 110.1)
- C2, C4: value 10u -> 22u
- moved J3 82.0 mm to (106.1, 144.5), turned to 0 degrees
- moved R17 49.1 mm to (134.5, 145.0)
- moved C29 48.4 mm to (131.8, 145.0)
- moved Q1 46.1 mm to (107.8, 137.3), turned to 90 degrees
- moved R13 40.3 mm to (125.1, 103.5)
- moved TP32 40.1 mm to (125.9, 89.6)
- moved D9 39.2 mm to (130.3, 88.6), turned to 180 degrees
- moved TP5 38.8 mm to (124.3, 91.1), turned to 180 degrees
- moved L2 38.5 mm to (129.5, 97.1)
- moved C6 35.5 mm to (126.8, 91.4), turned to 0 degrees
- moved C8 34.8 mm to (130.2, 91.4), turned to 0 degrees
- moved D1 30.5 mm to (119.7, 92.0)
- moved U2 30.5 mm to (124.0, 95.0)
- moved C11 30.5 mm to (116.8, 101.0)
- moved C13 30.5 mm to (116.8, 103.8)
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Routing:
- net GND: track 349.0 -> 0.28 mm, vias 27 -> 12
- net VBUS: track 103.9 -> 38.2 mm, vias 1 -> 0
- net UMB_~{ON}: track 63.1 -> 33.8 mm, vias 2 -> 0
- net /Power/VUMB: track 64.6 -> 38.6 mm, vias 1 -> 0
- net Net-(D11-K): track 37.5 -> 13.3 mm
- net Net-(D10-K): track 35.2 -> 12.7 mm, vias 1 -> 0
- net CANL: track 27.3 -> 45.9 mm
- net Net-(Q1-G): track 50.4 -> 33.1 mm
- net Net-(U1-INT1): track 30.8 -> 14.3 mm
- net BATT_READ: track 31.6 -> 15.2 mm, vias 0 -> 2
- net CANH: track 26.4 -> 39.3 mm
- net +3.3V: track 140.1 -> 151.9 mm, vias 4 -> 3
- net Net-(U2-CSP): track 23.4 -> 12.7 mm, vias 2 -> 0
- net Net-(D9-K): track 19.1 -> 8.89 mm
- net +BATT: track 117.7 -> 107.9 mm
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- added copper zone on F.Cu, net (none)
- added copper zone on F.Cu, net +3.3V
- added copper zone on F.Cu, net +BATT
- added copper zone on F.Cu, net VBUS

Commit message: Rev for review 4.25.2025
Parts:
- moved J10 43.1 mm to (96.7, 144.1)
- moved R15 41.7 mm to (101.8, 139.4), turned to 90 degrees
- moved C16 39.7 mm to (103.6, 139.3), turned to 90 degrees
- moved TP7 38.3 mm to (108.6, 148.8)
- moved R14 30.9 mm to (101.8, 142.5)
- moved C29 28.6 mm to (103.3, 142.5)
- moved R17 23.1 mm to (112.8, 137.2), turned to 0 degrees
- moved TP1 14.2 mm to (130.0, 82.5)
- moved R36 12.4 mm to (138.3, 86.1), turned to 90 degrees
- moved C26 9.76 mm to (140.9, 86.3), turned to 90 degrees
- moved TP2 9.39 mm to (130.0, 79.1)
- moved J2 6.72 mm to (143.3, 94.6)
- moved J8 5.51 mm to (145.9, 80.4)
- moved R35 4.00 mm to (143.5, 86.2), turned to -90 degrees
- moved J1 3.39 mm to (126.8, 80.4)
Routing:
- net Net-(Q1-G): track 33.1 -> 12.8 mm, vias 2 -> 0
- net CANL: track 45.9 -> 28.4 mm
- net CANH: track 39.3 -> 27.9 mm
- net Net-(J2-Pin_1): track 36.1 -> 27.9 mm
- net +BATT: track 107.9 -> 106.1 mm
- net Net-(C26-Pad1): track 4.24 -> 5.65 mm
- net /Power/ARM-OUT: track 5.75 -> 6.99 mm
- net /Power/VUMB: track 38.6 -> 37.8 mm
- net Net-(U2-CSP): track 12.7 -> 13.3 mm
