File: pcb/rcs-controller.kicad_pcb (KiCad board)
At the start: 2 copper layers, 45.6 x 73 mm, 100 parts, among them J1 00222-32051, J10 0022-232021, J2 0022-232021, J3 0022-232041, J4 Screw_Terminal_4_P3.50mm, J5 USB_C_Receptacle_USB2.0_14P, J6 Conn_01x03, J8 00222-32051, Q1 SI7465DP-T1-E3, Q2 SI7465DP-T1-E3, Q3 SI7465DP-T1-E3, Q4 PMV45EN2, Q5 PMV45EN2, SW1 SW_Push, U1 LSM6DSOX, U2 MP26123DR-LF-Z, U3 TPS63070, U4 ESP32-S3-WROOM-1

Commit message: More DRC cleanup, polishing, sticthing. Should be good to go.
Parts:
- moved D2 0.11 mm to (104.6, 118.4)
- moved R5 0.10 mm to (106.1, 118.4)
Routing:
- net +3.3V: track 95.7 -> 93.2 mm
- net Net-(Q5-G): track 40.9 -> 39.2 mm
- net Net-(D9-K): track 8.81 -> 9.70 mm
- net VBUS: track 36.2 -> 35.5 mm, vias 2 -> 4
- net /Power/VUMB: track 56.6 -> 55.9 mm
- net Net-(U3-L2): track 4.37 -> 5.00 mm
- net Net-(U3-L1): track 4.37 -> 5.00 mm
- net CANL: track 58.5 -> 57.9 mm
- net Net-(C26-Pad1): track 5.13 -> 5.70 mm
- net GND: vias 23 -> 130
- added copper zone on F.Cu, net +3.3V
Other:
- board text added: "${ISSUE_DATE}"
- board text added: "RCS"
- board text added: "V${REVISION}"
- board text removed: "Roll Control System Controller Board"
- board text removed: "V${REVISION} ${ISSUE_DATE}"
